File: hardware/HW/BuddiesJewel.sch (KiCad schematic (older format))
At the start: 25 parts, among them CON1 AVR-ISP6, CON2 ANTENNE, IC1 ATTINY25-P, P1 ALIM, U1 PT, U2 PT, U3 PT, U4 PT, U5 RF430CL330H

Commit message: change "RGB_LED (4)" D2 connector to "EXT_LED (3)" change ATtiny/RF430/WS2812/CON1 connections
Parts:
- removed D2: RGB_LED, ~, symbol RGB_LED
- removed JP2: JUMPER, ~, symbol JUMPER
- removed R7, R8: R, ~, symbol R
- added D2: EXT_LED, ~, symbol EXT_LED
- C1: value C -> 1 µF
- C2: value C -> 0,1 µF
- C3: value C -> 0,47 µF
- C4: value C -> 22 pF
- R1, R2, R3: value R -> not equipped
- R4, R5, R6: value R -> zero R
Connections:
- net +3.3V: now also D1.5 (VDD), D2.1 (VCC); no longer D1.6 (VSS)
- net GND: now also D1.6 (VSS), U5.10 (SCK), U5.9 (SCMS//CS), D2.3 (GND); no longer D1.5 (VDD)
- net IT/RST renamed RST
- net RST: no longer U5.8 (INTO)
- net PWM0/MISO renamed IT/MISO
- net IT/MISO: now also U5.8 (INTO); no longer JP1.2
- net PWM1: no longer names the net of IC1.2 (PB3(XTAL1/CLKI/OC1B/ADC3/PCINT3))
- net PWM2 renamed LED_DI
- net LED_DI: now also JP1.2, D2.2 (DI)
